File: mainboards/ESP32DK/kicad/mainboard.kicad_sch (KiCad schematic)
At the start: 9 parts

Commit message: Adding BOM for main board.
Parts:
- EB1, EB3, EB4: value ~ -> FE15-1; Manufacturer (none) -> Sullins Connector Solutions; Mfg Part # (none) -> PPTC151LFBN-RC; Substitution (none) -> Yes; Type (none) -> through hole
- EB2, EB5, ESP32L1, ESP32R1: Manufacturer (none) -> Sullins Connector Solutions; Mfg Part # (none) -> PPTC151LFBN-RC; Substitution (none) -> Yes; Type (none) -> through hole
- PWR1, RST1: Manufacturer (none) -> JST; Mfg Part # (none) -> B2B-XH-A; Substitution (none) -> No; Type (none) -> through hole
